File: Design/H00R8.brd (EAGLE design)
At the start: 34.6 x 30 mm, 1 part, among them P1 HEXABIT_17.32

Commit message: -Remove the module PN from the silkscreen -Update the schematic logo
Other:
- board text removed: "H00R80"
