File: Design/H00R8.sch (EAGLE design)
At the start: 1 part, among them P1 HEXABIT_17.32

Commit message: -Remove the module PN from the silkscreen -Update the schematic logo
Other:
- note added: "H00R8"
- note added: "H00R8_Frontend"
- note removed: "0"
- note removed: "H00R80"
- note removed: "H00R80_Frontend"
